Commit message: Project 4 - Map My World: exclude large rtabmap.db, link in README

File: my_robot/urdf/my_robot.xacro (robot description, xacro)
@@ -141,4 +141,11 @@
     <axis xyz="0 1 0" rpy="0 0 0"/>
   </joint>
+  <!-- Camera Optical Frame -->
+<joint type="fixed" name="camera_optical_joint">
+  <origin xyz="0 0 0" rpy="-1.5708 0 -1.5708"/>
+  <parent link="camera"/>
+  <child link="camera_link_optical"/>
+</joint>
+<link name="camera_link_optical"/>
   <!-- Hokuyo Lidar -->
   <link name="hokuyo">
